Commit message: 빌드 성공 및 런치 성공

File: description/ros2_control/ros2_control.xacro (robot description, xacro)
@@ -16,2 +16,3 @@
         </joint>
     </ros2_control>
+</robot>

File: description/urdf/sfbot.description.urdf.xacro (robot description, xacro)
@@ -1,5 +1,5 @@
 <?xml version='1.0' encoding='utf-8'?>
 <robot xmlns:xacro="http://www.ros.org/wiki/xacro" name="sfbot">
-    <link name="world" /link>
+    <link name="world" />
     <joint name="base_joint" type="fixed">
         <origin xyz="1.5 1.0 0" rpy="0 0 0"/>
@@ -16,5 +16,5 @@
             <origin xyz="0.0 0.0 0.0" rpy="0.0 0.0 0.0" />
             <geometry>
-                <mesh filename="package://my_robot_hardware/urdf/meshes/base_link.stl" scale="0.001 0.001 0.001" />
+                <mesh filename="package://sfbot_can/description/urdf/meshes/base_link.stl" scale="0.001 0.001 0.001" />
             </geometry>
         </visual>
@@ -22,5 +22,5 @@
             <origin xyz="0.0 0.0 0.0" rpy="0.0 0.0 0.0" />
             <geometry>
-                <mesh filename="package://my_robot_hardware/urdf/meshes/base_link.stl" scale="0.001 0.001 0.001" />
+                <mesh filename="package://sfbot_can/description/urdf/meshes/base_link.stl" scale="0.001 0.001 0.001" />
             </geometry>
         </collision>
@@ -35,5 +35,5 @@
             <origin xyz="-0.06300000093876953 9.933979985053653e-18 -1.058454243043459e-16" rpy="1.5707963267947935 1.5283000565118283 1.5707963267947935" />
             <geometry>
-                <mesh filename="package://my_robot_hardware/description/urdf/meshes/Component2.stl" scale="0.001 0.001 0.001" />
+                <mesh filename="package://sfbot_can/description/urdf/meshes/Component2.stl" scale="0.001 0.001 0.001" />
             </geometry>
         </visual>
@@ -41,5 +41,5 @@
             <origin xyz="-0.06300000093876953 9.933979985053653e-18 -1.058454243043459e-16" rpy="1.5707963267947935 1.5283000565118283 1.5707963267947935" />
             <geometry>
-                <mesh filename="package://my_robot_hardware/urdf/meshes/Component2.stl" scale="0.001 0.001 0.001" />
+                <mesh filename="package://sfbot_can/description/urdf/meshes/Component2.stl" scale="0.001 0.001 0.001" />
             </geometry>
         </collision>
@@ -54,5 +54,5 @@
             <origin xyz="-1.3108966917960693e-16 -1.242785109918427e-17 -0.08500000126659525" rpy="-3.797673495120442e-16 -4.476643978342218e-15 -3.099096383306725" />
             <geometry>
-                <mesh filename="package://my_robot_hardware/description/urdf/meshes/Component3.stl" scale="0.001 0.001 0.001" />
+                <mesh filename="package://sfbot_can/description/urdf/meshes/Component3.stl" scale="0.001 0.001 0.001" />
             </geometry>
         </visual>
@@ -60,5 +60,5 @@
             <origin xyz="-1.3108966917960693e-16 -1.242785109918427e-17 -0.08500000126659525" rpy="-3.797673495120442e-16 -4.476643978342218e-15 -3.099096383306725" />
             <geometry>
-                <mesh filename="package://my_robot_hardware/description/urdf/meshes/Component3.stl" scale="0.001 0.001 0.001" />
+                <mesh filename="package://sfbot_can/description/urdf/meshes/Component3.stl" scale="0.001 0.001 0.001" />
             </geometry>
         </collision>
@@ -73,5 +73,5 @@
             <origin xyz="0.013882699999999628 -0.026594559999999927 0.10326725730081326" rpy="3.1415926535897927 6.881253629370109e-15 3.099096383306725" />
             <geometry>
-                <mesh filename="package://my_robot_hardware/description/urdf/meshes/Component4.stl" scale="0.001 0.001 0.001" />
+                <mesh filename="package://sfbot_can/description/urdf/meshes/Component4.stl" scale="0.001 0.001 0.001" />
             </geometry>
         </visual>
@@ -79,5 +79,5 @@
             <origin xyz="0.013882699999999628 -0.026594559999999927 0.10326725730081326" rpy="3.1415926535897927 6.881253629370109e-15 3.099096383306725" />
             <geometry>
-                <mesh filename="package://my_robot_hardware/description/urdf/meshes/Component4.stl" scale="0.001 0.001 0.001" />
+                <mesh filename="package://sfbot_can/description/urdf/meshes/Component4.stl" scale="0.001 0.001 0.001" />
             </geometry>
         </collision>
@@ -92,5 +92,5 @@
             <origin xyz="-0.15112264860497968 0.023513786425360186 0.035483063201822256" rpy="2.952570499959834 1.3427262874177526 2.957353884887777" />
             <geometry>
-                <mesh filename="package://my_robot_hardware/description/urdf/meshes/Component5.stl" scale="0.001 0.001 0.001" />
+                <mesh filename="package://sfbot_can/description/urdf/meshes/Component5.stl" scale="0.001 0.001 0.001" />
             </geometry>
         </visual>
@@ -98,5 +98,5 @@
             <origin xyz="-0.15112264860497968 0.023513786425360186 0.035483063201822256" rpy="2.952570499959834 1.3427262874177526 2.957353884887777" />
             <geometry>
-                <mesh filename="package://my_robot_hardware/description/urdf/meshes/Component5.stl" scale="0.001 0.001 0.001" />
+                <mesh filename="package://sfbot_can/description/urdf/meshes/Component5.stl" scale="0.001 0.001 0.001" />
             </geometry>
         </collision>
@@ -111,5 +111,5 @@
             <origin xyz="-0.1602672573008139 4.5346505506138615e-09 -7.916735501878325e-10" rpy="-1.570796326795061 -1.5283000565118345 -1.5707963267947436" />
             <geometry>
-                <mesh filename="package://my_robot_hardware/description/urdf/meshes/Component6.stl" scale="0.001 0.001 0.001" />
+                <mesh filename="package://sfbot_can/description/urdf/meshes/Component6.stl" scale="0.001 0.001 0.001" />
             </geometry>
         </visual>
@@ -117,5 +117,5 @@
             <origin xyz="-0.1602672573008139 4.5346505506138615e-09 -7.916735501878325e-10" rpy="-1.570796326795061 -1.5283000565118345 -1.5707963267947436" />
             <geometry>
-                <mesh filename="package://my_robot_hardware/description/urdf/meshes/Component6.stl" scale="0.001 0.001 0.001" />
+                <mesh filename="package://sfbot_can/description/urdf/meshes/Component6.stl" scale="0.001 0.001 0.001" />
             </geometry>
         </collision>
@@ -130,5 +130,5 @@
             <origin xyz="-4.884981308350689e-17 0.0 -0.011199999999999996" rpy="-0.0 1.5707963267948923 0" />
             <geometry>
-                <mesh filename="package://my_robot_hardware/description/urdf/meshes/ak60-1-v1.stl" scale="0.001 0.001 0.001" />
+                <mesh filename="package://sfbot_can/description/urdf/meshes/ak60-1-v1.stl" scale="0.001 0.001 0.001" />
             </geometry>
         </visual>
@@ -136,5 +136,5 @@
             <origin xyz="-4.884981308350689e-17 0.0 -0.011199999999999996" rpy="-0.0 1.5707963267948923 0" />
             <geometry>
-                <mesh filename="package://my_robot_hardware/description/urdf/meshes/ak60-1-v1.stl" scale="0.001 0.001 0.001" />
+                <mesh filename="package://sfbot_can/description/urdf/meshes/ak60-1-v1.stl" scale="0.001 0.001 0.001" />
             </geometry>
         </collision>
@@ -149,5 +149,5 @@
             <origin xyz="0.0018629057736697058 -1.9984014443252818e-14 -0.04381050376250973" rpy="1.5707963267949068 1.5283000565118277 1.7143410555958367e-14" />
             <geometry>
-                <mesh filename="package://my_robot_hardware/description/urdf/meshes/ak60-2-v1.stl" scale="0.001 0.001 0.001" />
+                <mesh filename="package://sfbot_can/description/urdf/meshes/ak60-2-v1.stl" scale="0.001 0.001 0.001" />
             </geometry>
         </visual>
@@ -155,5 +155,5 @@
             <origin xyz="0.0018629057736697058 -1.9984014443252818e-14 -0.04381050376250973" rpy="1.5707963267949068 1.5283000565118277 1.7143410555958367e-14" />
             <geometry>
-                <mesh filename="package://my_robot_hardware/description/urdf/meshes/ak60-2-v1.stl" scale="0.001 0.001 0.001" />
+                <mesh filename="package://sfbot_can/description/urdf/meshes/ak60-2-v1.stl" scale="0.001 0.001 0.001" />
             </geometry>
         </collision>

File: description/urdf/sfbot.urdf.xacro (robot description, xacro)
@@ -1,5 +1,5 @@
 <?xml version="1.0"?>
 <robot xmlns:xacro="http://www.ros.org/wiki/xacro"  name="sfbot">
-    <xacro:include filename="$(find sfbot_can)/urdf/sfbot.urdf.xacro" />
-    <xacro:include filename="$(find sfbot_can)/ros2_control.xacro" />
+    <xacro:include filename="$(find sfbot_can)/description/urdf/sfbot.description.urdf.xacro" />
+    <xacro:include filename="$(find sfbot_can)/description/ros2_control/ros2_control.xacro" />
 </robot>

Commit message: 구동 성공

File: description/ros2_control/ros2_control.xacro (robot description, xacro)
@@ -9,8 +9,4 @@
             <state_interface name="position"/>
         </joint>
-        <joint name="ak70-10-v1_2_continuous-9">
-            <command_interface name="position"/>
-            <state_interface name="position"/>
-        </joint>
     </ros2_control>
 </robot>

Commit message: 2축 로봇팔 원점 설정 성공

File: description/ros2_control/ros2_control.xacro (robot description, xacro)
@@ -9,4 +9,8 @@
             <state_interface name="position"/>
         </joint>
+        <joint name="ak70-10-v1_2_continuous-9">
+            <command_interface name="position"/>
+            <state_interface name="position"/>
+        </joint>
     </ros2_control>
 </robot>
