Commit message: mesh 불러오기 성공

File: description/ros2_control/ros2_control_my_robot.xacro (robot description, xacro)
@@ -9,5 +9,4 @@
             <command_interface name="position"/>
             <state_interface name="position"/>
-            <state_interface name="velocity"/>
         </joint>
         <!-- Joint 2: Shoulder pitch (X-axis) -->
@@ -15,5 +14,4 @@
             <command_interface name="position"/>
             <state_interface name="position"/>
-            <state_interface name="velocity"/>
         </joint>
         <!-- Joint 3: Elbow rotation (Z-axis) -->
@@ -21,5 +19,4 @@
             <command_interface name="position"/>
             <state_interface name="position"/>
-            <state_interface name="velocity"/>
         </joint>
         <!-- Joint 4: Wrist pitch (X-axis) -->
@@ -27,5 +24,4 @@
             <command_interface name="position"/>
             <state_interface name="position"/>
-            <state_interface name="velocity"/>
         </joint>
         <!-- Joint 5: Wrist rotation (Z-axis) -->
@@ -33,5 +29,4 @@
             <command_interface name="position"/>
             <state_interface name="position"/>
-            <state_interface name="velocity"/>
         </joint>
         <!-- Joint 6: End effector rotation (X-axis) -->
@@ -39,5 +34,4 @@
             <command_interface name="position"/>
             <state_interface name="position"/>
-            <state_interface name="velocity"/>
         </joint>
     </ros2_control>

File: description/urdf/my_robot.description.urdf.xacro (robot description, xacro)
@@ -33,5 +33,5 @@
   <xacro:property name="joint_upper_limit" value="3.14"/>
   <!-- Macro for mesh link -->
-  <xacro:macro name="mesh_link" params="name mesh_file material_name collision_xyz:='0 0 0' visual_xyz:='0 0 0' collision_geometry:='' *collision_geometry_block">
+  <xacro:macro name="mesh_link" params="name mesh_file material_name collision_xyz:='0 0 0' visual_xyz:='0 0 0' collision_geometry:=''">
     <link name="${name}">
       <collision name="mesh_${name}_collision">
@@ -39,9 +39,10 @@
         <geometry>
           <xacro:if value="${collision_geometry == ''}">
-            <mesh filename="../meshes/stl/${mesh_file}" scale="${mesh_scale}"/>
+            <mesh filename="package://sfbot_can/description/urdf/meshes/${mesh_file}" scale="${mesh_scale}"/>
           </xacro:if>
-          <xacro:unless value="${collision_geometry == ''}">
-            <xacro:insert_block name="collision_geometry_block"/>
-          </xacro:unless>
+          <xacro:if value="${collision_geometry == 'box'}">
+            <box size="0.07 0.115 0.015"/>
+          </xacro:if>
+          <!-- 필요시 다른 geometry 타입들 추가 -->
         </geometry>
       </collision>
@@ -50,5 +51,5 @@
         <origin rpy="0.0 0.0 0.0" xyz="${visual_xyz}"/>
         <geometry>
-          <mesh filename="../meshes/stl/${mesh_file}" scale="${mesh_scale}"/>
+          <mesh filename="package://sfbot_can/description/urdf/meshes/${mesh_file}" scale="${mesh_scale}"/>
         </geometry>
       </visual>
@@ -83,5 +84,5 @@
   <!-- Base Link -->
   <xacro:mesh_link name="base_link"
-                   mesh_file="1_my_robot v2_base_link_1_Body1.stl"
+                   mesh_file="mesh_base_link.stl"
                    material_name="robot_black"
                    collision_xyz="0 0 0"
@@ -94,5 +95,5 @@
                      rpy="0 0 0"/>
   <xacro:mesh_link name="link1_motor"
-                   mesh_file="1_my_robot v2_link1_motor_1_Body1.stl"
+                   mesh_file="mesh_link1_motor.stl"
                    material_name="robot_red"
                    collision_xyz="0 0 -0.0263"
@@ -106,10 +107,8 @@
                         axis="0 0 1"/>
   <xacro:mesh_link name="link1_1"
-                   mesh_file="1_my_robot v2_link1_1_1_Body1.stl"
+                   mesh_file="mesh_link1_1.stl"
                    material_name="robot_blue"
                    collision_xyz="0 0 0.0075"
-                   visual_xyz="0 0 -0.077"
-                   collision_geometry="box">
-    <box size="0.07 0.115 0.015"/>
+                   visual_xyz="0 0 -0.077">
   </xacro:mesh_link>
   <!-- Link 1_2 -->
@@ -120,5 +119,5 @@
                      rpy="0 0 0"/>
   <xacro:mesh_link name="link1_2"
-                   mesh_file="1_my_robot v2_link1_2_1_Body2.stl"
+                   mesh_file="mesh_link1_2.stl"
                    material_name="robot_white"
                    collision_xyz="0 0 -0.092"
@@ -131,5 +130,5 @@
                      rpy="0 0 0"/>
   <xacro:mesh_link name="link2_motor"
-                   mesh_file="1_my_robot v2_link2_motor_1_Body1.stl"
+                   mesh_file="mesh_link2_motor.stl"
                    material_name="robot_red"
                    collision_xyz="0 0 -0.151"
@@ -143,5 +142,5 @@
                         axis="1 0 0"/>
   <xacro:mesh_link name="link2_1"
-                   mesh_file="1_my_robot v2_link2_1_1_Body1.stl"
+                   mesh_file="mesh_link2_1.stl"
                    material_name="robot_green"
                    collision_xyz="-0.009 0 -0.151"
@@ -154,5 +153,5 @@
                      rpy="0 0 0"/>
   <xacro:mesh_link name="link2_2"
-                   mesh_file="1_my_robot v2_link2_PLA_1_Body1.stl"
+                   mesh_file="mesh_link2_PLA.stl"
                    material_name="robot_white"
                    collision_xyz="-0.024 0 -0.151"
@@ -165,5 +164,5 @@
                      rpy="0 0 0"/>
   <xacro:mesh_link name="link2_3"
-                   mesh_file="1_my_robot v2_link2_7_1_Body1.stl"
+                   mesh_file="mesh_link2_7.stl"
                    material_name="robot_yellow"
                    collision_xyz="-0.099 0 -0.281"
@@ -176,5 +175,5 @@
                      rpy="0 0 0"/>
   <xacro:mesh_link name="link3_motor"
-                   mesh_file="1_my_robot v2_link3_motor_1_Body1.stl"
+                   mesh_file="mesh_link3_motor.stl"
                    material_name="robot_red"
                    collision_xyz="-0.099 0 -0.302"
@@ -188,5 +187,5 @@
                         axis="0 0 1"/>
   <xacro:mesh_link name="link3_1"
-                   mesh_file="1_my_robot v2_link3_1_1_Body1.stl"
+                   mesh_file="mesh_link3_1.stl"
                    material_name="robot_orange"
                    collision_xyz="-0.099 0 -0.34105"
@@ -199,5 +198,5 @@
                      rpy="0 0 0"/>
   <xacro:mesh_link name="link3_2"
-                   mesh_file="1_my_robot v2_link3_2_1_Body1.stl"
+                   mesh_file="mesh_link3_2.stl"
                    material_name="robot_purple"
                    collision_xyz="-0.099 0 -0.35605"
@@ -210,5 +209,5 @@
                      rpy="0 0 0"/>
   <xacro:mesh_link name="link4_motor"
-                   mesh_file="1_my_robot v2_link4_motor_1_Body1.stl"
+                   mesh_file="mesh_link4_motor.stl"
                    material_name="robot_red"
                    collision_xyz="-0.103 0 -0.41065"
@@ -222,10 +221,10 @@
                         axis="-1 0 0"/>
   <xacro:mesh_link name="link4_1"
-                   mesh_file="1_my_robot v2_link4_1_1_Body1.stl"
+                   mesh_file="mesh_link4_1.stl"
                    material_name="robot_blue"
                    collision_xyz="-0.0965 0 -0.41065"
                    visual_xyz="-0.0965 0 -0.41065"/>
   <!-- Link 4_2 -->
-  <xacro:fixed_joint name="link4_1.000_joint"
+  <xacro:fixed_joint name="link4_2_joint"
                      parent="link4_1"
                      child="link4_2"
@@ -233,5 +232,5 @@
                      rpy="0 0 0"/>
   <xacro:mesh_link name="link4_2"
-                   mesh_file="1_my_robot v2_link4_PLA_1_Body1.stl"
+                   mesh_file="mesh_link4_PLA.stl"
                    material_name="robot_white"
                    collision_xyz="-0.0815 0 -0.41065"
@@ -244,5 +243,5 @@
                      rpy="0 0 0"/>
   <xacro:mesh_link name="link4_3"
-                   mesh_file="1_my_robot v2_link4_7_1_Body1.stl"
+                   mesh_file="mesh_link4_7.stl"
                    material_name="robot_green"
                    collision_xyz="-0.0065 0 -0.51065"
@@ -255,5 +254,5 @@
                      rpy="0 0 0"/>
   <xacro:mesh_link name="link5_motor"
-                   mesh_file="1_my_robot v2_link5_motor_1_Body1.stl"
+                   mesh_file="mesh_link5_motor.stl"
                    material_name="robot_red"
                    collision_xyz="-0.0065 0 -0.53065"
@@ -267,5 +266,5 @@
                         axis="0 0 1"/>
   <xacro:mesh_link name="link5_1"
-                   mesh_file="1_my_robot v2_link5_1_1_Body1.stl"
+                   mesh_file="mesh_link5_1.stl"
                    material_name="robot_yellow"
                    collision_xyz="-0.0065 0 -0.55965"
@@ -278,5 +277,5 @@
                      rpy="0 0 0"/>
   <xacro:mesh_link name="link5_2"
-                   mesh_file="1_my_robot v2_link5_2_1_Body2.stl"
+                   mesh_file="mesh_link5_2.stl"
                    material_name="robot_orange"
                    collision_xyz="-0.0065 0 -0.57965"
@@ -289,5 +288,5 @@
                      rpy="0 0 0"/>
   <xacro:mesh_link name="link6_motor"
-                   mesh_file="1_my_robot v2_link6_motor_1_Body1.stl"
+                   mesh_file="mesh_link6_motor.stl"
                    material_name="robot_red"
                    collision_xyz="-0.01 0 -0.62915"
@@ -301,5 +300,5 @@
                         axis="1 0 0"/>
   <xacro:mesh_link name="link6_1"
-                   mesh_file="1_my_robot v2_link6_1_1_Body1.stl"
+                   mesh_file="mesh_link6_1.stl"
                    material_name="robot_purple"
                    collision_xyz="-0.012 0 -0.62915"

File: description/urdf/my_robot.urdf.xacro (robot description, xacro)
@@ -1,5 +1,5 @@
 <?xml version="1.0"?>
 <robot xmlns:xacro="http://www.ros.org/wiki/xacro"  name="my_robot">
-    <xacro:include filename="$(find sfbot_can)/description/ros2_control/ros2_control_test.xacro" />
+    <xacro:include filename="$(find sfbot_can)/description/ros2_control/ros2_control_my_robot.xacro" />
     <xacro:include filename="$(find sfbot_can)/description/urdf/my_robot.description.urdf.xacro" />
 </robot>
