Commit message: 충돌 삭제

File: description/urdf/sfbot.description.urdf_collision.xacro (robot description, xacro)
@@ -19,4 +19,10 @@
             </geometry>
         </visual>
+        <collision name="base_link_collision">
+            <origin xyz="0.0 0.0 0.0" rpy="0.0 0.0 0.0" />
+            <geometry>
+                <mesh filename="package://sfbot_can/description/urdf/meshes/base_link.stl" scale="0.001 0.001 0.001" />
+            </geometry>
+        </collision>
     </link>
     <link name="Component2">
@@ -32,4 +38,10 @@
             </geometry>
         </visual>
+        <collision name="Component2_collision">
+            <origin xyz="-0.06300000093876953 9.933979985053653e-18 -1.058454243043459e-16" rpy="1.5707963267947935 1.5283000565118283 1.5707963267947935" />
+            <geometry>
+                <mesh filename="package://sfbot_can/description/urdf/meshes/Component2.stl" scale="0.001 0.001 0.001" />
+            </geometry>
+        </collision>
     </link>
     <link name="Component3">
@@ -45,4 +57,10 @@
             </geometry>
         </visual>
+        <collision name="Component3_collision">
+            <origin xyz="-1.3108966917960693e-16 -1.242785109918427e-17 -0.08500000126659525" rpy="-3.797673495120442e-16 -4.476643978342218e-15 -3.099096383306725" />
+            <geometry>
+                <mesh filename="package://sfbot_can/description/urdf/meshes/Component3.stl" scale="0.001 0.001 0.001" />
+            </geometry>
+        </collision>
     </link>
     <link name="Component4">
@@ -58,4 +76,10 @@
             </geometry>
         </visual>
+        <collision name="Component4_collision">
+            <origin xyz="0.013882699999999628 -0.026594559999999927 0.10326725730081326" rpy="3.1415926535897927 6.881253629370109e-15 3.099096383306725" />
+            <geometry>
+                <mesh filename="package://sfbot_can/description/urdf/meshes/Component4.stl" scale="0.001 0.001 0.001" />
+            </geometry>
+        </collision>
     </link>
     <link name="Component5">
@@ -71,4 +95,10 @@
             </geometry>
         </visual>
+        <collision name="Component5_collision">
+            <origin xyz="-0.15112264860497968 0.023513786425360186 0.035483063201822256" rpy="2.952570499959834 1.3427262874177526 2.957353884887777" />
+            <geometry>
+                <mesh filename="package://sfbot_can/description/urdf/meshes/Component5.stl" scale="0.001 0.001 0.001" />
+            </geometry>
+        </collision>
     </link>
     <link name="Component6">
@@ -84,4 +114,10 @@
             </geometry>
         </visual>
+        <collision name="Component6_collision">
+            <origin xyz="-0.1602672573008139 4.5346505506138615e-09 -7.916735501878325e-10" rpy="-1.570796326795061 -1.5283000565118345 -1.5707963267947436" />
+            <geometry>
+                <mesh filename="package://sfbot_can/description/urdf/meshes/Component6.stl" scale="0.001 0.001 0.001" />
+            </geometry>
+        </collision>
     </link>
     <link name="ak70-10-v1_1">
@@ -97,4 +133,10 @@
             </geometry>
         </visual>
+        <collision name="ak70-10-v1_1_collision">
+            <origin xyz="-4.884981308350689e-17 0.0 -0.011199999999999996" rpy="-0.0 1.5707963267948923 0" />
+            <geometry>
+                <mesh filename="package://sfbot_can/description/urdf/meshes/ak70-1-v1.stl" scale="0.001 0.001 0.001" />
+            </geometry>
+        </collision>
     </link>
     <link name="ak70-10-v1_2">
@@ -110,4 +152,10 @@
             </geometry>
         </visual>
+        <collision name="ak70-10-v1_2_collision">
+            <origin xyz="0.0018629057736697058 -1.9984014443252818e-14 -0.04381050376250973" rpy="1.5707963267949068 1.5283000565118277 1.7143410555958367e-14" />
+            <geometry>
+                <mesh filename="package://sfbot_can/description/urdf/meshes/ak70-2-v1.stl" scale="0.001 0.001 0.001" />
+            </geometry>
+        </collision>
     </link>
     <joint name="base_link_fixed-4" type="fixed">
