Commit message: 6개모터 적용 성공

File: description/urdf/test.description.urdf.xacro (robot description, xacro)
@@ -31,5 +31,5 @@
                 <box size="0.05 0.05 0.05"/>
             </geometry>
-            <material name="white"/>
+            <material name="orange"/>
         </visual>
         <collision>

File: description/urdf/test.urdf.xacro (robot description, xacro)
@@ -1,5 +1,5 @@
 <?xml version="1.0"?>
 <robot xmlns:xacro="http://www.ros.org/wiki/xacro"  name="test">
+    <xacro:include filename="$(find sfbot_can)/description/ros2_control/ros2_control_test.xacro" />
     <xacro:include filename="$(find sfbot_can)/description/urdf/test.description.urdf.xacro" />
-    <xacro:include filename="$(find sfbot_can)/description/ros2_control/ros2_control_test.xacro" />
 </robot>

Commit message: 다중 CAN 통신 인터페이스 추가 및 rviz 런치 추가

File: description/urdf/test.description.urdf.xacro (robot description, xacro)
@@ -88,5 +88,5 @@
         <parent link="link_1"/>
         <child link="link_2"/>
-        <axis xyz="0 1 0"/>
+        <axis xyz="1 0 0"/>
         <limit lower="-3.14" upper="3.14" effort="100" velocity="1"/>
     </joint>
@@ -136,5 +136,5 @@
         <parent link="link_3"/>
         <child link="link_4"/>
-        <axis xyz="0 1 0"/>
+        <axis xyz="1 0 0"/>
         <limit lower="-3.14" upper="3.14" effort="100" velocity="1"/>
     </joint>
@@ -184,5 +184,5 @@
         <parent link="link_5"/>
         <child link="link_6"/>
-        <axis xyz="0 1 0"/>
+        <axis xyz="1 0 0"/>
         <limit lower="-3.14" upper="3.14" effort="100" velocity="1"/>
     </joint>
